File: jubileev2.kicad_pcb (KiCad board)
At the start: 2 copper layers, 75.4 x 75.3 mm, 42 parts, among them IC2 74HC14D,653, J1 PJ-202A, J3 LED_RING_PADS, Q1 UMH3N, Q3 PZT2222A, SW3 MAIN_BUTTON, U1 AMS1117-3.3, U2 AMS1117-5.0, U3 CH340C

Commit message: Update PCB with new USB-C PD power supply
Parts:
- removed D2: D_Schottky, Diode_SMD:D_SOD-123
- removed D3: D, Diode_SMD:D_SOD-123
- removed G***: LOGO, jubileev2:roundel_ss
- removed J1: PJ-202A, digikey-footprints:Barrel_Jack_5.5mmODx2.1mmID_PJ-202A
- added C13: 10uF, Capacitor_SMD:C_0805_2012Metric, F.Cu at (62.5, 112.6)
- added C7: 0.1uF, Capacitor_SMD:C_0805_2012Metric, F.Cu at (106.5, 111.0)
- added D6: D_Small, Diode_SMD:D_SOD-123, F.Cu at (56.4, 121.9)
- added Q2: AO3400A, Package_TO_SOT_SMD:SOT-23, F.Cu at (90.2, 104.2)
- added U4: IP2721, Package_SO:TSSOP-16_4.4x5mm_P0.65mm, F.Cu at (100.0, 104.6)
- added U5: 78D09LL-TN3-R, Package_TO_SOT_SMD:TO-252-2, F.Cu at (67.5, 119.1)
- moved C2 9.82 mm to (56.4, 116.0)
- moved F1 5.50 mm to (106.5, 104.5), turned to -90 degrees
- moved R4 3.05 mm to (112.0, 84.4)
- moved R3 2.83 mm to (112.1, 104.7)
Connections:
- net Net-(R3-Pad2) renamed CC1
- net Net-(R4-Pad2) renamed CC2
- ANT1 pad 11: (no net) -> unconnected-(ANT1-IO26-Pad11)
- ANT1 pad 12: (no net) -> unconnected-(ANT1-IO27-Pad12)
- ANT1 pad 13: (no net) -> unconnected-(ANT1-IO14-Pad13)
- ANT1 pad 14: (no net) -> unconnected-(ANT1-IO12-Pad14)
- ANT1 pad 16: (no net) -> unconnected-(ANT1-IO13-Pad16)
- ANT1 pad 17: (no net) -> unconnected-(ANT1-SD2-Pad17)
- ANT1 pad 18: (no net) -> unconnected-(ANT1-SD3-Pad18)
- ANT1 pad 19: (no net) -> unconnected-(ANT1-CMD-Pad19)
- ANT1 pad 20: (no net) -> unconnected-(ANT1-CLK-Pad20)
- ANT1 pad 21: (no net) -> unconnected-(ANT1-SD0-Pad21)
- ANT1 pad 22: (no net) -> unconnected-(ANT1-SD1-Pad22)
- ANT1 pad 23: (no net) -> unconnected-(ANT1-IO15-Pad23)
- ANT1 pad 24: (no net) -> unconnected-(ANT1-IO2-Pad24)
- ANT1 pad 26: (no net) -> unconnected-(ANT1-IO4-Pad26)
- ANT1 pad 27: (no net) -> unconnected-(ANT1-IO16-Pad27)
- ANT1 pad 28: (no net) -> unconnected-(ANT1-IO17-Pad28)
- ANT1 pad 29: (no net) -> unconnected-(ANT1-IO5-Pad29)
- ANT1 pad 30: (no net) -> unconnected-(ANT1-IO18-Pad30)
- ANT1 pad 31: (no net) -> unconnected-(ANT1-IO19-Pad31)
- ANT1 pad 32: (no net) -> unconnected-(ANT1-NC-Pad32)
- ANT1 pad 33: (no net) -> unconnected-(ANT1-IO21-Pad33)
- ANT1 pad 4: (no net) -> unconnected-(ANT1-SENSOR_VP-Pad4)
- ANT1 pad 5: (no net) -> unconnected-(ANT1-SENSOR_VN-Pad5)
- ANT1 pad 6: (no net) -> unconnected-(ANT1-IO34-Pad6)
- ANT1 pad 7: (no net) -> unconnected-(ANT1-IO35-Pad7)
- ANT1 pad 8: (no net) -> unconnected-(ANT1-IO32-Pad8)
- ANT1 pad 9: (no net) -> unconnected-(ANT1-IO33-Pad9)
- C2 pad 1: +9V -> +15V
- F1 pad 1: Net-(D3-Pad2) -> Net-(F1-Pad1)
- F1 pad 2: Net-(F1-Pad2) -> Net-(Q2-D)
- IC2 pad 10: (no net) -> unconnected-(IC2-5Y-Pad10)
- IC2 pad 11: (no net) -> unconnected-(IC2-5A-Pad11)
- IC2 pad 12: (no net) -> unconnected-(IC2-6Y-Pad12)
- IC2 pad 13: (no net) -> unconnected-(IC2-6A-Pad13)
- IC2 pad 3: (no net) -> unconnected-(IC2-2A-Pad3)
- IC2 pad 4: (no net) -> unconnected-(IC2-2Y-Pad4)
- IC2 pad 5: (no net) -> unconnected-(IC2-3A-Pad5)
- IC2 pad 6: (no net) -> unconnected-(IC2-3Y-Pad6)
- IC2 pad 8: (no net) -> unconnected-(IC2-4Y-Pad8)
- IC2 pad 9: (no net) -> unconnected-(IC2-4A-Pad9)
- U2 pad 3: +9V -> +15V
- U3 pad 10: (no net) -> unconnected-(U3-~{DSR}-Pad10)
- U3 pad 11: (no net) -> unconnected-(U3-~{RI}-Pad11)
- U3 pad 12: (no net) -> unconnected-(U3-~{DCD}-Pad12)
- U3 pad 15: (no net) -> unconnected-(U3-R232-Pad15)
- U3 pad 2: ESP_RXD -> ESP_TXD
- U3 pad 3: ESP_TXD -> ESP_RXD
- U3 pad 7: (no net) -> unconnected-(U3-NC-Pad7)
- U3 pad 8: (no net) -> unconnected-(U3-NC-Pad8)
- U3 pad 9: (no net) -> unconnected-(U3-~{CTS}-Pad9)
- USB1 pad 11: Net-(F1-Pad2) -> Net-(F1-Pad1)
- USB1 pad 2: Net-(F1-Pad2) -> Net-(F1-Pad1)
- USB1 pad 3: (no net) -> unconnected-(USB1-SBU2-Pad3)
- USB1 pad 9: (no net) -> unconnected-(USB1-SBU1-Pad9)
Routing:
- net +15V: track 0.00 -> 80.5 mm
- net +5V: track 59.4 -> 15.4 mm
- net CC2: track 6.66 -> 41.5 mm, vias 0 -> 2
- net Net-(Q2-D): track 0.00 -> 24.9 mm, vias 0 -> 2
- net Net-(F1-Pad2): track 22.0 -> 0.00 mm, vias 2 -> 0
- net CC1: track 7.05 -> 25.6 mm, vias 0 -> 2
- net Net-(F1-Pad1): track 0.00 -> 15.3 mm, vias 0 -> 2
- net GND: track 68.6 -> 79.7 mm, vias 20 -> 25
- net Net-(D2-Pad2): track 8.65 -> 0.00 mm
- net Net-(Q2-G): track 0.00 -> 8.28 mm
- net Net-(D6-A): track 0.00 -> 4.62 mm
- net +9V: track 70.8 -> 74.7 mm
- net Net-(D3-Pad2): track 3.68 -> 0.00 mm
- net ESP_TXD: track 31.7 -> 28.5 mm
- net Net-(U3-UD+): track 22.7 -> 21.7 mm
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Other:
- outline, holes or cut-outs redrawn
- net class Default removed
- board text added: "1996 Stock / Jubilee Line Door Button Replacement PCB"
- board text added: "Will Furnell - willfurnell.com Hugh Wells - crablab.uk"
- board text added: "r5-2"
- board text removed: "-"
- board text removed: "CENTRE POSITIVE"
- board text removed: "Jubilee Line Door Button replacement PCB"
- board text removed: "Will Furnell 2021 willfurnell.com"
- board text removed: "r4"
